Commit message: Renamed robo_bin_picking_gym dir to robo_ml_gym

File: robo_ml_gym/models/irb120/irb120.urdf (robot description, URDF)
Before this commit: robot irb120, 7 links, 6 joints
Links:
- link base_link: geometry collision mesh filename=robo_ml_gym/models/irb120/collision/base_link.stl; visual mesh filename=robo_ml_gym/models/irb120/visual/base_link.stl
- link link_1: geometry collision mesh filename=robo_ml_gym/models/irb120/collision/link_1.stl; visual mesh filename=robo_ml_gym/models/irb120/visual/link_1.stl
- link link_2: geometry collision mesh filename=robo_ml_gym/models/irb120/collision/link_2.stl; visual mesh filename=robo_ml_gym/models/irb120/visual/link_2.stl
- link link_3: geometry collision mesh filename=robo_ml_gym/models/irb120/collision/link_3.stl; visual mesh filename=robo_ml_gym/models/irb120/visual/link_3.stl
- link link_4: geometry collision mesh filename=robo_ml_gym/models/irb120/collision/link_4.stl; visual mesh filename=robo_ml_gym/models/irb120/visual/link_4.stl
- link link_5: geometry collision mesh filename=robo_ml_gym/models/irb120/collision/link_5.stl; visual mesh filename=robo_ml_gym/models/irb120/visual/link_5.stl
- link link_6: geometry collision mesh filename=robo_ml_gym/models/irb120/collision/link_6_ef.stl; visual mesh filename=robo_ml_gym/models/irb120/visual/link_6_ef.stl

Commit message: fixed distance from ef to cube, cube can be held

File: robo_ml_gym/models/irb120/irb120.urdf (robot description, URDF)
Before this commit: robot irb120, 7 links, 6 joints
Links:
- added link link_7, mass 0.0136784407912; collision mesh filename=robo_ml_gym/models/irb120/collision/link_7_ef.stl; visual mesh filename=robo_ml_gym/models/irb120/visual/link_7_ef.stl
- link link_6: geometry collision mesh filename=robo_ml_gym/models/irb120/collision/link_6_ef_short.stl; visual mesh filename=robo_ml_gym/models/irb120/visual/link_6_ef_short.stl
Joints:
- added joint joint_7: type fixed, parent link_6, child link_7, origin xyz=0.223 0 0 rpy=0 0 0, axis 1 0 0, limit lower=-6.98132 upper=6.98132 effort=0 velocity=7.33038

Commit message: Use correct end effector location in distances

File: robo_ml_gym/models/irb120/irb120.urdf (robot description, URDF)
Before this commit: robot irb120, 8 links, 7 joints
Joints:
- joint joint_7: limit lower=-6.98132 upper=6.98132 effort=0 velocity=7.33038 -> lower=0 upper=0 effort=0 velocity=0
